File: Driver_High.kicad_sch (KiCad schematic)
At the start: 19 parts, among them Q901 DMP3099-x, U901 FODM217A, U902 UCC21222DR

Commit message: Initial commit micro-inverter
Signed-off-by: Jean Alinei <jean.alinei@owntech.org>
Parts:
- added D501, D502: STPS0520Z, Diode_SMD:D_SOD-323, symbol Device:D
- added RGH501, RGL501: 2,2, Resistor_SMD:R_0805_2012Metric, symbol Device:R
- added RpdH501, RpdL501: 1k, Resistor_SMD:R_0805_2012Metric, symbol Device:R
- renumbered C902 to C904, C903 to C906, C904 to C908, C905 to C910, C906 to C911, C907 to C913, C908 to C915, C909 to C917, D901 to D902, Q901 to Q902, R901 to R902, R902 to R904, R903 to R905, R904 to R908, R905 to R909, R906 to R912, U901 to U902, U902 to U904
Connections:
- net DGND: no longer U904.5 (DIS)
- net GNDREF: now also RpdL501.1
- net PWM_H: now also D501.2 (A), RGH501.2, RpdH501.2; no longer U904.15 (OUTA)
- net PWM_L: now also D502.2 (A), RGL501.2, RpdL501.2; no longer U904.10 (OUTB)
- net SW_Node: now also RpdH501.1
- new net DIS: U904.5 (DIS)
- new net Drive_H: D501.1 (K), RGH501.1, U904.15 (OUTA)
- new net Drive_L: D502.1 (K), RGL501.1, U904.10 (OUTB)
Other:
- note removed: "Decoupling GATE driver"
- title: (none) -> Micro-inverter - 400W
- moved on the sheet: C901, C904, C906, C908, C910, C911, C913, C915, C917, D902, Q902, R902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
