File: Flyback.kicad_sch (KiCad schematic)
At the start: 88 parts, among them J5001 B2B-EH-A(LF)(SN), J5002 B2B-EH-A(LF)(SN), J5003 Header_2_54_01x03, Q5001 DMN10H220L-7, Q5002 TK13P25D,RQ, T5001 PA2467NL, U1001 AZ1117CH-5.0TRG1, U5001 MCP6486UT-E/LT, U5002 AZ1117CH-5.0TRG1, U5003 NCP12700ADNR2G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

Commit message: Initial commit micro-inverter
Signed-off-by: Jean Alinei <jean.alinei@owntech.org>
Parts:
- C5016, C5022: value 100pF -> 100pF
- C5026: value 1nF -> 1nF
- U5001: value MCP6486UT-E/LT -> MCP6486UT-E/LT
