File: feeder.kicad_sch (KiCad schematic)
At the start: 12 parts, among them U601 MCP1799T-5002H/TT, U602 MCP1799T-5002H/TT, U603 MCP1799T-5002H/TT

Commit message: Initial commit micro-inverter
Signed-off-by: Jean Alinei <jean.alinei@owntech.org>
Parts:
- U601, U602, U603: value MCP1799T-5002H/TT -> MCP1799T-5002H/TT
Other:
- title: Feeders -> Micro-inverter - 400W
