File: high_voltage_bridge.kicad_sch (KiCad schematic)
At the start: 46 parts, among them Q501 IPD60R210PFD7SAUMA1, Q502 IPD60R210PFD7SAUMA1, Q503 IPD60R210PFD7SAUMA1, Q504 IPD60R210PFD7SAUMA1, U501 AMC1202DWVR, U502 AMC1311BDWVR, U503 MCP6486UT-E/LT, U504 MCP6486UT-E/LT

Commit message: Initial commit micro-inverter
Signed-off-by: Jean Alinei <jean.alinei@owntech.org>
Parts:
- removed C3, C4: 100nF, Capacitor_SMD:C_1210_3225Metric, symbol Device:C
- removed C511, C512: 10uF, Footprints:C_Rect_L31.5mm_W13.0mm_P27.50mm_MKS4, symbol Device:C
- removed D501, D502, D503, D504: STPS0520Z, Diode_SMD:D_SOD-323, symbol Device:D
- removed Q501, Q502, Q503, Q504: IPD60R210PFD7SAUMA1, Package_TO_SOT_SMD:TO-252-2, symbol Transistor_FET:QM6006D
- removed RGH501, RGH502, RGL501, RGL502: 2,2, Resistor_SMD:R_0805_2012Metric, symbol Device:R
- removed RpdH501, RpdH502, RpdL501, RpdL502: 1k, Resistor_SMD:R_0805_2012Metric, symbol Device:R
- removed Rv501, Rv502, Rv503, Rv504: 1M, Resistor_SMD:R_0805_2012Metric, symbol Device:R_Small
- removed Rv505: 16K, Resistor_SMD:R_0805_2012Metric, symbol Device:R_Small
- U503, U504: value MCP6486UT-E/LT -> MCP6486UT-E/LT
Connections:
- net GNDREF: no longer R514.2, U501.3 (VINN)
- net I_{IIHigh_P}: no longer R514.1
- new net I_{IIHigh_N}: U501.3 (VINN)
Other:
- removed sheet Driver2
- removed sheet Driver3
