File: low_voltage_bridge.kicad_sch (KiCad schematic)
At the start: 55 parts, among them Q301 IPD200N15N3GATMA1, Q302 IPD200N15N3GATMA1, Q303 IPD200N15N3GATMA1, Q304 IPD200N15N3GATMA1, U301 +-20A Hall, U302 AMC1311BDWVR, U303 MCP6486UT-E/LT, U304 MCP6486UT-E/LT

Commit message: Initial commit micro-inverter
Signed-off-by: Jean Alinei <jean.alinei@owntech.org>
Parts:
- removed C301, C302, C316, C323: 100nF, Capacitor_SMD:C_1206_3216Metric, symbol Device:C_Small
- removed C305, C322: 20pF, Footprints:C_0805_2012Metric, symbol Device:C_Small
- removed R301, R302, R303, R304: 27k, Footprints:R_0805_2012Metric, symbol Device:R_Small
- removed R307, R310: 5.9k, Footprints:R_0805_2012Metric, symbol Device:R_Small
- removed R308, R309: 20k, Footprints:R_0805_2012Metric, symbol Device:R_Small
- removed U302: AMC1311BDWVR, Package_SO:SOIC-8_7.5x5.85mm_P1.27mm, symbol Symbols:AMC1311DBW
- removed U303, U304: MCP6486UT-E/LT, Package_TO_SOT_SMD:SOT-353_SC-70-5_Handsoldering, symbol Symbols:MCP6486UT-E/LT
- Q301, Q302, Q303, Q304: value IPD200N15N3GATMA1 -> IPD200N15N3GATMA1
Connections:
- net GND renamed V_{IHigh}_{GND}_{-}
- net V_{IHigh}_{GND}_{-}: no longer C1.2, C2.2, Q302.3 (S), Q304.3 (S), RpdL301.1, RpdL302.1
- new net: C2.2, Q304.3 (S), RpdL302.1
Other:
- note removed: "At 0 ampere ILow is equal to 0.5xVCC = 2.5V so V_{SHIFTED} = 1V (amplitude: 0 to 2048 mV)"
- note removed: "Circuit can be seen as non inverting opamp with gain : G = 1+(RC/RD) and a potential on non-inverting input equal to : V+ =(VOUTP-VOUTN)*(RA/(RA+RB)) V_{Diff} = (VOUTP-VOUTN) V+ = V_{Diff}*(RA/(RA+RB)) V+ = V_{Diff}*(27k/(27k+27k)) V+ = V_{Diff}*0.5"
- note removed: "DIGITAL AREA"
- note removed: "Low side current conditioning"
- note removed: "Low side voltage conditioning"
- note removed: "POWER AREA"
- note removed: "RA"
- note removed: "RB"
- note removed: "RC"
- note removed: "RD"
- note removed: "RE"
- note removed: "RF"
- note removed: "RG"
- note removed: "RH"
- note removed: "Simulation available https://tinyurl.com/ym6es7vl"
- note removed: "Simulation available https://tinyurl.com/yodepbhp"
- note removed: "V_{SHIFTED} = G*V+ V_{SHIFTED} = [1+(RC/RD)]*0.5*V_{Diff} V_{SHIFTED} = [1+(27k/27k)]*0.5*V_{Diff} V_{SHIFTED} = 2*0.5*V_{Diff} V_{SHIFTED} = V_{Diff}"
- note removed: "V_{SHIFTED} = [((RE + RF)*RH) / ((RH + RG)*RF)] * I_{Low} - [(RE/RF)* 5V_{Digital}] V_{SHIFTED} = [((5.9k + 20k)*20k) / ((20k + 5.9k)*20k)] * I_{Low} - [(5.9k/20k)* 5] ** If RH = RF and RE = RG, gain is unity V_{SHIFTED} = I_{Low} - (5.9k/20k)* 5 V_{SHIFTED} = I_{Low} - 1.5V"
- note removed: "https://www.allegromicro.com/en/ Insights-and-Innovations/ Technical-Documents/ Hall-Effect-Sensor-IC-Publications/ Shifting-the-Offset -Voltage-of-Current-Sensors"
