File: KiCAD_Files/low_side_voltage.kicad_sch (KiCad schematic)
At the start: 15 parts, among them U311 AMC1311BDWVR, U312 MCP6486UT-E/LT

Commit message: Change the repo structure to match standard tree.
Signed-off-by: Jean Alinei <jean.alinei@owntech.org>
Parts:
- renumbered C340 to C301, C341 to C302, C342 to C305, C343 to C316, R327 to R301, R328 to R302, R329 to R303, R330 to R304, Rv526 to Rv501, Rv527 to Rv502, Rv528 to Rv503, Rv529 to Rv504, Rv530 to Rv505, U311 to U302, U312 to U303
Changed lines of the file:
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@@
 		(on_board yes)
 		(dnp no)
-		(property "Reference" "#PWR0344"
+		(property "Reference" "#PWR0303"
 			(at 55.88 107.95 0)
 			(effects
@@
 		)
 		(instances
-			(project "DAB"
+			(project "micro_inverter"
 				(path "/741fe409-f733-4088-8b5c-1042510db0b9/3ea151e7-6bb7-4df0-80a5-b2ad4a7f2d78"
 					(reference "#PWR0303")
@@
 		(on_board yes)
 		(dnp no)
-		(property "Reference" "C341"
+		(property "Reference" "C302"
 			(at 95.25 68.58 0)
 			(effects
@@
 		)
 		(instances
-			(project "DAB"
+			(project "micro_inverter"
 				(path "/741fe409-f733-4088-8b5c-1042510db0b9/3ea151e7-6bb7-4df0-80a5-b2ad4a7f2d78"
 					(reference "C302")
@@
 		(on_board yes)
 		(dnp no)
-		(property "Reference" "#PWR027"
+		(property "Reference" "#PWR07"
 			(at 119.38 83.82 0)
 			(effects
@@
 		)
 		(instances
-			(project "DAB"
+			(project "micro_inverter"
 				(path "/741fe409-f733-4088-8b5c-1042510db0b9/3ea151e7-6bb7-4df0-80a5-b2ad4a7f2d78"
 					(reference "#PWR07")
@@
 		(dnp no)
 		(fields_autoplaced yes)
-		(property "Reference" "#PWR0347"
+		(property "Reference" "#PWR0308"
 			(at 131.318 63.5 90)
 			(effects
@@
 		)
 		(instances
-			(project "DAB"
+			(project "micro_inverter"
 				(path "/741fe409-f733-4088-8b5c-1042510db0b9/3ea151e7-6bb7-4df0-80a5-b2ad4a7f2d78"
 					(reference "#PWR0308")
@@
 		(on_board yes)
 		(dnp no)
-		(property "Reference" "#PWR026"
+		(property "Reference" "#PWR06"
 			(at 92.71 81.28 0)
 			(effects
@@
 		)
 		(instances
-			(project "DAB"
+			(project "micro_inverter"
 				(path "/741fe409-f733-4088-8b5c-1042510db0b9/3ea151e7-6bb7-4df0-80a5-b2ad4a7f2d78"
 					(reference "#PWR06")
@@
 		(on_board yes)
 		(dnp no)
-		(property "Reference" "U312"
+		(property "Reference" "U303"
 			(at 134.62 82.55 0)
 			(effects
@@
 		)
 		(instances
-			(project "DAB"
+			(project "micro_inverter"
 				(path "/741fe409-f733-4088-8b5c-1042510db0b9/3ea151e7-6bb7-4df0-80a5-b2ad4a7f2d78"
 					(reference "U303")
@@
 		(dnp no)
 		(fields_autoplaced yes)
-		(property "Reference" "#PWR0346"
+		(property "Reference" "#PWR0306"
 			(at 94.488 62.23 90)
 			(effects
@@
 		)
 		(instances
-			(project "DAB"
+			(project "micro_inverter"
 				(path "/741fe409-f733-4088-8b5c-1042510db0b9/3ea151e7-6bb7-4df0-80a5-b2ad4a7f2d78"
 					(reference "#PWR0306")
@@
 		(on_board yes)
 		(dnp no)
-		(property "Reference" "R328"
+		(property "Reference" "R302"
 			(at 104.14 94.488 90)
 			(effects
@@
 		)
 		(instances
-			(project "DAB"
+			(project "micro_inverter"
 				(path "/741fe409-f733-4088-8b5c-1042510db0b9/3ea151e7-6bb7-4df0-80a5-b2ad4a7f2d78"
 					(reference "R302")
@@
 		(on_board yes)
 		(dnp no)
-		(property "Reference" "Rv528"
+		(property "Reference" "Rv503"
 			(at 34.5186 71.2216 0)
 			(effects
@@
 		)
 		(instances
-			(project "DAB"
+			(project "micro_inverter"
 				(path "/741fe409-f733-4088-8b5c-1042510db0b9/3ea151e7-6bb7-4df0-80a5-b2ad4a7f2d78"
 					(reference "Rv503")
@@
 		(on_board yes)
 		(dnp no)
-		(property "Reference" "#PWR029"
+		(property "Reference" "#PWR010"
 			(at 140.97 83.82 0)
 			(effects
@@
 		)
 		(instances
-			(project "DAB"
+			(project "micro_inverter"
 				(path "/741fe409-f733-4088-8b5c-1042510db0b9/3ea151e7-6bb7-4df0-80a5-b2ad4a7f2d78"
 					(reference "#PWR010")
@@
 		(on_board yes)
 		(dnp no)
-		(property "Reference" "R329"
+		(property "Reference" "R303"
 			(at 114.3 77.978 0)
 			(effects
@@
 		)
 		(instances
-			(project "DAB"
+			(project "micro_inverter"
 				(path "/741fe409-f733-4088-8b5c-1042510db0b9/3ea151e7-6bb7-4df0-80a5-b2ad4a7f2d78"
 					(reference "R303")
@@
 		(on_board yes)
 		(dnp no)
-		(property "Reference" "#PWR0343"
+		(property "Reference" "#PWR0302"
 			(at 54.61 81.28 0)
 			(effects
@@
 		)
 		(instances
-			(project "DAB"
+			(project "micro_inverter"
 				(path "/741fe409-f733-4088-8b5c-1042510db0b9/3ea151e7-6bb7-4df0-80a5-b2ad4a7f2d78"
 					(reference "#PWR0302")
@@
 		(on_board yes)
 		(dnp no)
-		(property "Reference" "#PWR028"
+		(property "Reference" "#PWR09"
 			(at 129.54 104.14 0)
 			(effects
@@
 		)
 		(instances
-			(project "DAB"
+			(project "micro_inverter"
 				(path "/741fe409-f733-4088-8b5c-1042510db0b9/3ea151e7-6bb7-4df0-80a5-b2ad4a7f2d78"
 					(reference "#PWR09")
@@
 		(on_board yes)
 		(dnp no)
-		(property "Reference" "C343"
+		(property "Reference" "C316"
 			(at 133.096 72.644 0)
 			(effects
@@
 		)
 		(instances
-			(project "DAB"
+			(project "micro_inverter"
 				(path "/741fe409-f733-4088-8b5c-1042510db0b9/3ea151e7-6bb7-4df0-80a5-b2ad4a7f2d78"
 					(reference "C316")
@@
 		(on_board yes)
 		(dnp no)
-		(property "Reference" "R330"
+		(property "Reference" "R304"
 			(at 132.08 107.696 90)
 			(effects
@@
 		)
 		(instances
-			(project "DAB"
+			(project "micro_inverter"
 				(path "/741fe409-f733-4088-8b5c-1042510db0b9/3ea151e7-6bb7-4df0-80a5-b2ad4a7f2d78"
 					(reference "R304")
@@
 		(on_board yes)
 		(dnp no)
-		(property "Reference" "#PWR025"
+		(property "Reference" "#PWR04"
 			(at 91.44 107.95 0)
 			(effects
@@
 		)
 		(instances
-			(project "DAB"
+			(project "micro_inverter"
 				(path "/741fe409-f733-4088-8b5c-1042510db0b9/3ea151e7-6bb7-4df0-80a5-b2ad4a7f2d78"
 					(reference "#PWR04")
@@
 		(on_board yes)
 		(dnp no)
-		(property "Reference" "Rv529"
+		(property "Reference" "Rv504"
 			(at 34.5186 78.8416 0)
 			(effects
@@
 		)
 		(instances
-			(project "DAB"
+			(project "micro_inverter"
 				(path "/741fe409-f733-4088-8b5c-1042510db0b9/3ea151e7-6bb7-4df0-80a5-b2ad4a7f2d78"
 					(reference "Rv504")
@@
 		(on_board yes)
 		(dnp no)
-		(property "Reference" "U311"
+		(property "Reference" "U302"
 			(at 61.468 75.184 0)
 			(effects
@@
 		)
 		(instances
-			(project "DAB"
+			(project "micro_inverter"
 				(path "/741fe409-f733-4088-8b5c-1042510db0b9/3ea151e7-6bb7-4df0-80a5-b2ad4a7f2d78"
 					(reference "U302")
@@
 		(on_board yes)
 		(dnp no)
-		(property "Reference" "C342"
+		(property "Reference" "C305"
 			(at 132.08 118.872 90)
 			(effects
@@
 		)
 		(instances
-			(project "DAB"
+			(project "micro_inverter"
 				(path "/741fe409-f733-4088-8b5c-1042510db0b9/3ea151e7-6bb7-4df0-80a5-b2ad4a7f2d78"
 					(reference "C305")
@@
 		(on_board yes)
 		(dnp no)
-		(property "Reference" "Rv530"
+		(property "Reference" "Rv505"
 			(at 34.5186 90.2716 0)
 			(effects
@@
 		)
 		(instances
-			(project "DAB"
+			(project "micro_inverter"
 				(path "/741fe409-f733-4088-8b5c-1042510db0b9/3ea151e7-6bb7-4df0-80a5-b2ad4a7f2d78"
 					(reference "Rv505")
@@
 		(on_board yes)
 		(dnp no)
-		(property "Reference" "Rv527"
+		(property "Reference" "Rv502"
 			(at 34.5186 63.6016 0)
 			(effects
@@
 		)
 		(instances
-			(project "DAB"
+			(project "micro_inverter"
 				(path "/741fe409-f733-4088-8b5c-1042510db0b9/3ea151e7-6bb7-4df0-80a5-b2ad4a7f2d78"
 					(reference "Rv502")
@@
 		(on_board yes)
 		(dnp no)
-		(property "Reference" "C340"
+		(property "Reference" "C301"
 			(at 52.07 68.58 0)
 			(effects
@@
 		)
 		(instances
-			(project "DAB"
+			(project "micro_inverter"
 				(path "/741fe409-f733-4088-8b5c-1042510db0b9/3ea151e7-6bb7-4df0-80a5-b2ad4a7f2d78"
 					(reference "C301")
@@
 		(dnp no)
 		(fields_autoplaced yes)
-		(property "Reference" "#PWR0345"
+		(property "Reference" "#PWR0304"
 			(at 60.198 62.23 90)
 			(effects
@@
 		)
 		(instances
-			(project "DAB"
+			(project "micro_inverter"
 				(path "/741fe409-f733-4088-8b5c-1042510db0b9/3ea151e7-6bb7-4df0-80a5-b2ad4a7f2d78"
 					(reference "#PWR0304")
@@
 		(on_board yes)
 		(dnp no)
-		(property "Reference" "R327"
+		(property "Reference" "R301"
 			(at 103.886 81.534 90)
 			(effects
@@
 		)
 		(instances
-			(project "DAB"
+			(project "micro_inverter"
 				(path "/741fe409-f733-4088-8b5c-1042510db0b9/3ea151e7-6bb7-4df0-80a5-b2ad4a7f2d78"
 					(reference "R301")
@@
 		(on_board yes)
 		(dnp no)
-		(property "Reference" "Rv526"
+		(property "Reference" "Rv501"
 			(at 34.5186 55.9816 0)
 			(effects
@@
 		)
 		(instances
-			(project "DAB"
+			(project "micro_inverter"
 				(path "/741fe409-f733-4088-8b5c-1042510db0b9/3ea151e7-6bb7-4df0-80a5-b2ad4a7f2d78"
 					(reference "Rv501")
