File: KiCAD_Files/micro_inverter.kicad_sch (KiCad schematic)
At the start: 47 parts, among them J1 Conn_01x01, J103 B2B-EH-A(LF)(SN), J104 B2B-EH-A(LF)(SN), J105 B2B-EH-A(LF)(SN), J2 Conn_01x01, J3 Conn_01x01, J7 Conn_01x01, J8 Conn_01x01, K1 G2RL-1A-H, K2 G2RL-2A, Q501 IPD60R210PFD7SAUMA1, Q502 IPD60R210PFD7SAUMA1, Q503 IPD60R210PFD7SAUMA1, Q504 IPD60R210PFD7SAUMA1, Q505 IPD60R210PFD7SAUMA1, Q506 IPD60R210PFD7SAUMA1, Q507 IPD60R210PFD7SAUMA1, Q508 IPD60R210PFD7SAUMA1, Q509 IPD60R210PFD7SAUMA1, Q510 IPD60R210PFD7SAUMA1, Q511 IPD60R210PFD7SAUMA1, Q512 IPD60R210PFD7SAUMA1, T1 Transformer_1P_1S

Commit message: Change the repo structure to match standard tree.
Signed-off-by: Jean Alinei <jean.alinei@owntech.org>
Connections:
- net Driver4/PWM_H is gone; now on net Driver4/PWM_H: Q505.1 (G)
- net Driver4/PWM_L is gone; now on net Driver4/PWM_L: Q508.1 (G)
- net Driver4/SW_Node is gone; now on net Driver4/SW_Node: Q507.3 (S), Q508.2 (D), T1.1 (AA)
- net Driver5/PWM_H is gone; now on net Driver5/PWM_H: Q509.1 (G)
- net Driver5/PWM_L is gone; now on net Driver5/PWM_L: Q512.1 (G)
- net Driver5/SW_Node is gone; now on net Driver5/SW_Node: Q511.3 (S), Q512.2 (D), T1.4 (SB)
- net Driver4/PWM_H: no longer Q507.1 (G)
- net Driver4/PWM_L: no longer Q506.1 (G)
- net Driver4/SW_Node: no longer Q505.3 (S), Q506.2 (D), T1.2 (AB)
- net Driver5/PWM_H: no longer Q511.1 (G)
- net Driver5/PWM_L: no longer Q510.1 (G)
- net Driver5/SW_Node: no longer Q509.3 (S), Q510.2 (D), T1.3 (SA)
- new net Driver4/PWM_H: Q507.1 (G)
- new net Driver4/PWM_L: Q506.1 (G)
- new net Driver4/SW_Node: Q505.3 (S), Q506.2 (D), T1.2 (AB)
- new net Driver5/PWM_H: Q511.1 (G)
- new net Driver5/PWM_L: Q510.1 (G)
- new net Driver5/SW_Node: Q509.3 (S), Q510.2 (D), T1.3 (SA)
Other:
- sheet AC Voltage sense: file untitled.kicad_sch -> low_side_voltage.kicad_sch
- sheet DC Voltage sense: file untitled.kicad_sch -> low_side_voltage.kicad_sch
- sheet Grid Voltage sense: file untitled.kicad_sch -> low_side_voltage.kicad_sch
Changed lines of the file:
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@@
 			)
 		)
-		(property "Sheetfile" "untitled.kicad_sch"
+		(property "Sheetfile" "low_side_voltage.kicad_sch"
 			(at 276.86 56.4646 0)
 			(effects
@@
 			)
 		)
-		(property "Sheetfile" "untitled.kicad_sch"
+		(property "Sheetfile" "low_side_voltage.kicad_sch"
 			(at 63.5 57.7346 0)
 			(effects
@@
 			)
 		)
-		(property "Sheetfile" "untitled.kicad_sch"
+		(property "Sheetfile" "low_side_voltage.kicad_sch"
 			(at 231.14 56.4646 0)
 			(effects
