File: KiCAD_Files/power.kicad_sch (KiCad schematic)
At the start: 170 parts, among them J1 Conn_01x01, J2 Conn_01x01, J3 Conn_01x01, J5 Conn_01x01, J8 Conn_01x01, K1 HF140FF/012-2HSWTF, Q1 CID12N65D, Q10 CJAC90SN12, Q11 ZXMN7A11GTA, Q2 CID12N65D, Q3 CID12N65D, Q4 CID12N65D, Q5 CJAC90SN12, Q6 CJAC90SN12, Q7 CJAC90SN12, Q8 CJAC90SN12, Q9 CJAC90SN12, T1 Transformer_1P_1S, T2 Transformer_1P_1S, U1 INA240A1PWR, U2 INA240A1PWR, U3 UCC27282DRC, U4 UCC27282DRC

Commit message: added on the schematic the changes andres sugested
Parts:
- added D10: 460V, Diode_SMD:D_SMF, symbol Diode:SMF51A
- added D6, D7: D_Schottky, symbol Device:D_Schottky
- added D8, D9: 100V, Diode_SMD:D_SMF, symbol Diode:SMF51A
- added R11, R6: 1M, symbol Device:R
- added R111, R112: 500m, Resistor_SMD:R_0603_1608Metric, symbol Device:R_Small
- Logo101: value ~ -> (none)
- R108, R109: now not fitted
Connections:
- net GND_{HV}: now also D10.2 (A2), R6.2
- net GND_{LV}: now also D6.2 (A), D7.2 (A), D8.2 (A2), D9.2 (A2)
- net HV_{BUS}: now also D10.1 (A1), R11.1
- net LSW1: now also R111.2; no longer C40.2, U3.5 (HS)
- net LSW2: now also R112.2; no longer C8.2, U4.5 (HS)
- net V_{IHigh1}: now also D8.1 (A1)
- net V_{IHigh2}: now also D9.1 (A1)
- new net: R11.2, R6.1
- new net: C8.2, D7.1 (K), R112.1, U4.5 (HS)
- new net: C40.2, D6.1 (K), R111.1, U3.5 (HS)
Other:
- note added: "Big voltage, multiple resistor for sharing voltage"
- note added: "ONLY compatible with DRC (DRP is another pinout)"
- note added: "Schottky to protect from negatives spikes"
- moved on the sheet: C136, C137, C40, C53, C8, C9, U3, U4
